Commit message: add spoon task

File: robo_manip_baselines/envs/assets/tacto/objects/grasp/cube.urdf (robot description, URDF)
Before this commit: robot cube, 1 links, 0 joints
Links:
- link baseLink: mass 1 -> 0.1; geometry collision mesh filename=meshes/cube.obj scale=.10 .05 .15; visual mesh filename=meshes/cube.obj scale=.10 .05 .15
